File: etch_a_sketch/etch_a_sketch.kicad_pcb (KiCad board)
At the start: 2 copper layers, 200 x 101.8 mm, 62 parts, among them J101 SAM_FTSH-107-01-L-DV-K-A_STDC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, J102 WE_61304021121, SW101 CK_GSPTS004003, SW102 ESW_RA11131121, U101 STM32L433CCT6, U102 TI_TPS2553DBVT, U103 ST_LIS2DW12TR, U104 MIC_MCP1253T-33X50I/MS, U105 MIC_MCP1253T-33X50I/MS

Commit message: BOM done
Parts:
- D101: value EE_EAST1616RGBB2 -> EAST1616RGBB2
Changed lines of the file:
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@@
 		(layer "F.Cu")
 		(at 120.995 124.585)
-		(descr "Mounting Hole 3.2mm, M3, generated by kicad-footprint-generator mountinghole.py")
-		(tags "mountinghole M3 ISO14580")
+		(descr "Mounting Hole 3.2mm, M3, ISO14580")
+		(tags "mounting hole 3.2mm m3 iso14580")
 		(property "Reference" "H103"
 			(at 0 -3.7 0)
@@
 			(layers "*.Cu" "*.Mask")
 			(remove_unused_layers no)
-			(zone_connect 2)
 		)
 		(pad "1" connect circle
@@
 			(size 5.5 5.5)
 			(layers "F.Cu" "F.Mask")
-			(zone_connect 2)
 		)
 		(pad "1" connect circle
@@
 			(size 5.5 5.5)
 			(layers "B.Cu" "B.Mask")
-			(zone_connect 2)
 		)
 		(embedded_fonts no)
@@
 		)
 		(embedded_fonts no)
-		(model "C:/Users/dhyey/Desktop/PCB 3D Models/MIC_MCP1253T-33X50IMS.step"
+		(model "${DHYEY_PROJECTS}/MIC_MCP1253T-33X50IMS.step"
 			(offset
 				(xyz 0 0 0)
@@
 		)
 		(embedded_fonts no)
-		(model "C:/Users/dhyey/Desktop/PCB 3D Models/STM32L433CCT6.STEP"
+		(model "${DHYEY_PROJECTS}/STM32L433CCT6.STEP"
 			(offset
 				(xyz 0 0 0.85)
@@
 		(layer "F.Cu")
 		(at 246 53.1)
-		(descr "Mounting Hole 3.2mm, M3, generated by kicad-footprint-generator mountinghole.py")
-		(tags "mountinghole M3 ISO14580")
+		(descr "Mounting Hole 3.2mm, M3, ISO14580")
+		(tags "mounting hole 3.2mm m3 iso14580")
 		(property "Reference" "H106"
 			(at 0 -3.7 0)
@@
 			(layers "*.Cu" "*.Mask")
 			(remove_unused_layers no)
-			(zone_connect 2)
 		)
 		(pad "1" connect circle
@@
 			(size 5.5 5.5)
 			(layers "F.Cu" "F.Mask")
-			(zone_connect 2)
 		)
 		(pad "1" connect circle
@@
 			(size 5.5 5.5)
 			(layers "B.Cu" "B.Mask")
-			(zone_connect 2)
 		)
 		(embedded_fonts no)
@@
 		(layer "F.Cu")
 		(at 179.005 75.385)
-		(descr "Mounting Hole 3.2mm, M3, generated by kicad-footprint-generator mountinghole.py")
-		(tags "mountinghole M3 ISO14580")
+		(descr "Mounting Hole 3.2mm, M3, ISO14580")
+		(tags "mounting hole 3.2mm m3 iso14580")
 		(property "Reference" "H102"
 			(at 0 -3.7 0)
@@
 			(layers "*.Cu" "*.Mask")
 			(remove_unused_layers no)
-			(zone_connect 2)
 		)
 		(pad "1" connect circle
@@
 			(size 5.5 5.5)
 			(layers "F.Cu" "F.Mask")
-			(zone_connect 2)
 		)
 		(pad "1" connect circle
@@
 			(size 5.5 5.5)
 			(layers "B.Cu" "B.Mask")
-			(zone_connect 2)
 		)
 		(embedded_fonts no)
@@
 		(layer "F.Cu")
 		(at 54 146.9)
-		(descr "Mounting Hole 3.2mm, M3, generated by kicad-footprint-generator mountinghole.py")
-		(tags "mountinghole M3 ISO14580")
+		(descr "Mounting Hole 3.2mm, M3, ISO14580")
+		(tags "mounting hole 3.2mm m3 iso14580")
 		(property "Reference" "H107"
 			(at 0 -3.7 0)
@@
 			(layers "*.Cu" "*.Mask")
 			(remove_unused_layers no)
-			(zone_connect 2)
 		)
 		(pad "1" connect circle
@@
 			(size 5.5 5.5)
 			(layers "F.Cu" "F.Mask")
-			(zone_connect 2)
 		)
 		(pad "1" connect circle
@@
 			(size 5.5 5.5)
 			(layers "B.Cu" "B.Mask")
-			(zone_connect 2)
 		)
 		(embedded_fonts no)
@@
 		(layer "F.Cu")
 		(at 120.995 75.385)
-		(descr "Mounting Hole 3.2mm, M3, generated by kicad-footprint-generator mountinghole.py")
-		(tags "mountinghole M3 ISO14580")
+		(descr "Mounting Hole 3.2mm, M3, ISO14580")
+		(tags "mounting hole 3.2mm m3 iso14580")
 		(property "Reference" "H101"
 			(at 0 -3.7 0)
@@
 			(layers "*.Cu" "*.Mask")
 			(remove_unused_layers no)
-			(zone_connect 2)
 		)
 		(pad "1" connect circle
@@
 			(size 5.5 5.5)
 			(layers "F.Cu" "F.Mask")
-			(zone_connect 2)
 		)
 		(pad "1" connect circle
@@
 			(size 5.5 5.5)
 			(layers "B.Cu" "B.Mask")
-			(zone_connect 2)
 		)
 		(embedded_fonts no)
@@
 		)
 		(embedded_fonts no)
-		(model "C:/Users/dhyey/Desktop/PCB 3D Models/TTE_P120PK-Y25BR10K.stp"
+		(model "${DHYEY_PROJECTS}/TTE_P120PK-Y25BR10K.stp"
 			(offset
 				(xyz -3.75 -7 0)
@@
 		)
 		(embedded_fonts no)
-		(model "C:/Users/dhyey/Desktop/PCB 3D Models/TI_TPS2553DBVT_SOT-23-6.STEP"
+		(model "${DHYEY_PROJECTS}/TI_TPS2553DBVT_SOT-23-6.STEP"
 			(offset
 				(xyz 0 0 0)
@@
 		)
 		(embedded_fonts no)
-		(model "C:/Users/dhyey/Desktop/PCB 3D Models/ESW_RA11131121.stp"
+		(model "${DHYEY_PROJECTS}/ESW_RA11131121.stp"
 			(offset
 				(xyz 0 -7 1.25)
@@
 		)
 		(embedded_fonts no)
-		(model "C:/Users/dhyey/Desktop/PCB 3D Models/MIC_MCP1253T-33X50IMS.step"
+		(model "${DHYEY_PROJECTS}/MIC_MCP1253T-33X50IMS.step"
 			(offset
 				(xyz 0 0 0)
@@
 		(layer "F.Cu")
 		(at 179.005 124.585)
-		(descr "Mounting Hole 3.2mm, M3, generated by kicad-footprint-generator mountinghole.py")
-		(tags "mountinghole M3 ISO14580")
+		(descr "Mounting Hole 3.2mm, M3, ISO14580")
+		(tags "mounting hole 3.2mm m3 iso14580")
 		(property "Reference" "H104"
 			(at 0 -3.7 0)
@@
 			(layers "*.Cu" "*.Mask")
 			(remove_unused_layers no)
-			(zone_connect 2)
 		)
 		(pad "1" connect circle
@@
 			(size 5.5 5.5)
 			(layers "F.Cu" "F.Mask")
-			(zone_connect 2)
 		)
 		(pad "1" connect circle
@@
 			(size 5.5 5.5)
 			(layers "B.Cu" "B.Mask")
-			(zone_connect 2)
 		)
 		(embedded_fonts no)
@@
 		)
 		(embedded_fonts no)
-		(model "C:/Users/dhyey/Desktop/PCB 3D Models/ST_LIS2DW12TR.step"
+		(model "${DHYEY_PROJECTS}/ST_LIS2DW12TR.step"
 			(offset
 				(xyz 0 0 0)
@@
 		(layer "F.Cu")
 		(at 54 53.1)
-		(descr "Mounting Hole 3.2mm, M3, generated by kicad-footprint-generator mountinghole.py")
-		(tags "mountinghole M3 ISO14580")
+		(descr "Mounting Hole 3.2mm, M3, ISO14580")
+		(tags "mounting hole 3.2mm m3 iso14580")
 		(property "Reference" "H105"
 			(at 0 -3.7 0)
@@
 			(layers "*.Cu" "*.Mask")
 			(remove_unused_layers no)
-			(zone_connect 2)
 		)
 		(pad "1" connect circle
@@
 			(size 5.5 5.5)
 			(layers "F.Cu" "F.Mask")
-			(zone_connect 2)
 		)
 		(pad "1" connect circle
@@
 			(size 5.5 5.5)
 			(layers "B.Cu" "B.Mask")
-			(zone_connect 2)
 		)
 		(embedded_fonts no)
@@
 		(layer "F.Cu")
 		(at 246 146.9)
-		(descr "Mounting Hole 3.2mm, M3, generated by kicad-footprint-generator mountinghole.py")
-		(tags "mountinghole M3 ISO14580")
+		(descr "Mounting Hole 3.2mm, M3, ISO14580")
+		(tags "mounting hole 3.2mm m3 iso14580")
 		(property "Reference" "H108"
 			(at 0 -3.7 0)
@@
 			(layers "*.Cu" "*.Mask")
 			(remove_unused_layers no)
-			(zone_connect 2)
 		)
 		(pad "1" connect circle
@@
 			(size 5.5 5.5)
 			(layers "F.Cu" "F.Mask")
-			(zone_connect 2)
 		)
 		(pad "1" connect circle
@@
 			(size 5.5 5.5)
 			(layers "B.Cu" "B.Mask")
-			(zone_connect 2)
 		)
 		(embedded_fonts no)
@@
 		)
 		(embedded_fonts no)
-		(model "C:/Users/dhyey/Desktop/PCB 3D Models/SAM_FTSH-107-01-L-DV-K-A_STDC14.stp"
+		(model "${DHYEY_PROJECTS}/SAM_FTSH-107-01-L-DV-K-A_STDC14.stp"
 			(offset
 				(xyz 0 0 0.45)
@@
 		)
 		(embedded_fonts no)
-		(model "C:/Users/dhyey/Desktop/PCB 3D Models/WE_61304021121.stp"
+		(model "${DHYEY_PROJECTS}/WE_61304021121.stp"
 			(offset
 				(xyz 0 -1.25 1.25)
@@
 		)
 		(embedded_fonts no)
-		(model "C:/Users/dhyey/Desktop/PCB 3D Models/CK_GSPTS004003.stp"
+		(model "${DHYEY_PROJECTS}/CK_GSPTS004003.stp"
 			(offset
 				(xyz 0 0 0)
@@
 		)
 		(embedded_fonts no)
-		(model "C:/Users/dhyey/Desktop/PCB 3D Models/TTE_P120PK-Y25BR10K.stp"
+		(model "${DHYEY_PROJECTS}/TTE_P120PK-Y25BR10K.stp"
 			(offset
 				(xyz -3.75 -7 0)
@@
 			)
 		)
-		(property "Value" "EE_EAST1616RGBB2"
+		(property "Value" "EAST1616RGBB2"
 			(at 0 0 0)
 			(unlocked yes)
@@
 		)
 		(embedded_fonts no)
-		(model "C:/Users/dhyey/Desktop/PCB 3D Models/EE_EAST1616RGBB2.STEP"
+		(model "${DHYEY_PROJECTS}/EE_EAST1616RGBB2.STEP"
 			(offset
 				(xyz 0 0 0)
@@
 		)
 		(embedded_fonts no)
-		(model "C:/Users/dhyey/Desktop/PCB 3D Models/KE_3034TR.step"
+		(model "${DHYEY_PROJECTS}/KE_3034TR.step"
 			(offset
 				(xyz 0 7.5 4)
